File: KiCAD/optode-alex/optode-alex.kicad_pcb (KiCad board)
At the start: 2 copper layers, 8.6 x 4.4 mm, 2 parts, among them J1 Conn_01x03

Commit message: as built gerbers, start software for testing
Other:
- board text added: "NN SRC v1.0"
Changed lines of the file:
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@@
 		(allow_soldermask_bridges_in_footprints no)
 		(pcbplotparams
-			(layerselection 0x0001000_7ffffffe)
+			(layerselection 0x00010f0_ffffffff)
 			(plot_on_all_layers_selection 0x0000000_00000000)
 			(disableapertmacros no)
@@
 			(sketchpadsonfab no)
 			(subtractmaskfromsilk no)
-			(outputformat 3)
+			(outputformat 1)
 			(mirror no)
 			(drillshape 0)
 			(scaleselection 1)
-			(outputdirectory "dxf/")
+			(outputdirectory "gerber/")
 		)
 	)
@@
 		(at 136.695 97.27)
 		(property "Reference" "D1"
-			(at 1.355 -1.72 0)
-			(unlocked yes)
-			(layer "F.SilkS")
+			(at 0.505 2.43 -0)
+			(unlocked yes)
+			(layer "B.SilkS")
 			(effects
 				(font
@@
 					(thickness 0.1)
 				)
+				(justify mirror)
 			)
 		)
@@
 		(tags "Through hole pin header THT 1x03 1.00mm single row")
 		(property "Reference" "J1"
-			(at 0 -1.56 0)
+			(at -2.1 0.95 0)
 			(layer "F.SilkS")
 			(effects
@@
 		(layer "Edge.Cuts")
 	)
+	(gr_text "NN SRC\nv1.0"
+		(at 142.1 100 0)
+		(layer "B.SilkS")
+		(effects
+			(font
+				(size 0.8128 0.8128)
+				(thickness 0.127)
+			)
+			(justify left bottom mirror)
+		)
+	)
 	(dimension
 		(type aligned)
@@
 		)
 		(height 2.2)
-		(gr_text "4.4000 mm"
+		(gr_text "0.1732 in"
 			(at 132.65 98.8 90)
 			(layer "User.2")
@@
 		(height 7.4)
 		(orientation 0)
-		(gr_text "2.4000 mm"
+		(gr_text "0.0945 in"
 			(at 143.4 107.15 0)
 			(layer "Cmts.User")
@@
 		(height 4.3)
 		(orientation 0)
-		(gr_text "3.3000 mm"
+		(gr_text "0.1299 in"
 			(at 140.55 104.15 0)
 			(layer "Cmts.User")
@@
 		(height 12.7)
 		(orientation 1)
-		(gr_text "2.5000 mm"
+		(gr_text "0.0984 in"
 			(at 150.45 98.85 90)
 			(layer "Cmts.User")
@@
 		(height 2.7)
 		(orientation 1)
-		(gr_text "4.1000 mm"
+		(gr_text "0.1614 in"
 			(at 146.15 98.85 90)
 			(layer "Cmts.User")
@@
 		(height -3.8)
 		(orientation 0)
-		(gr_text "8.6000 mm"
+		(gr_text "0.3386 in"
 			(at 140.3 91.65 0)
 			(layer "Cmts.User")
